File: kicad_files/simpleESP32/_autosave-simpleESP32.kicad_pcb (KiCad board)
At the start: 2 copper layers, 1 part, among them U1 ESP32-WROOM-32D

Commit message: progress with schematic
Parts:
- added J1: Conn_01x07, Connector_PinHeader_2.54mm:PinHeader_1x07_P2.54mm_Vertical, F.Cu at (137.2, 123.2)
- added J2: Conn_01x07, Connector_PinHeader_2.54mm:PinHeader_1x07_P2.54mm_Vertical, F.Cu at (151.1, 123.2)
- added J3: USB_B_Micro, Connector_USB:USB_Micro-B_Molex-105017-0001, F.Cu at (143.5, 143.5)
- added SW1: SW_SPST, Button_Switch_SMD:SW_SPST_B3U-1000P, F.Cu at (166.4, 130.8)
- added U2: FT231XS, Package_SO:SSOP-20_3.9x8.7mm_P0.635mm, F.Cu at (144.8, 130.8)
- moved U1 2.54 mm to (143.5, 108.0)
