File: kicad_files/simpleESP32/simpleESP32.sch (KiCad schematic (older format))
At the start: 4 parts, among them U1 ESP32-WROOM-32D

Commit message: added footprints
Parts:
- added SW?: SW_SPST, Button_Switch_SMD:SW_SPST_B3U-1000P, symbol Switch:SW_SPST
Changed lines of the file:
@@
+	1    0    0    -1
+$EndComp
+$Comp
+L Switch:SW_SPST SW?
+U 1 1 5E6A071C
+P 8500 4050
+F 0 "SW?" H 8500 4285 50  0000 C CNN
+F 1 "SW_SPST" H 8500 4194 50  0000 C CNN
+F 2 "Button_Switch_SMD:SW_SPST_B3U-1000P" H 8500 4050 50  0001 C CNN
+F 3 "~" H 8500 4050 50  0001 C CNN
+	1    8500 4050
 	1    0    0    -1
 $EndComp

Commit message: progress with schematic
Parts:
- added J1, J2: Conn_01x07, Connector_PinHeader_2.54mm:PinHeader_1x07_P2.54mm_Vertical, symbol Connector_Generic:Conn_01x07
- added R?: 10K, symbol Device:R
- gave numbers to parts that had none: 4
Connections:
- net labels added: +3.3V, +5V, DM, DP, GND, RXD, TXD
- wire segments 0 -> 25
Other:
- moved on the sheet: J3, SW1, U1, U2, U3

Commit message: schematic completed
Parts:
- added C1, C3: 10uF, Capacitor_SMD:C_0805_2012Metric, symbol Device:CP_Small
- added C2: 0.1uF, Capacitor_SMD:C_0805_2012Metric, symbol Device:CP_Small
- added SW2: EN, Button_Switch_SMD:SW_SPST_B3U-1000P, symbol Switch:SW_SPST
- R1: renamed from R?; footprint (none) -> Resistor_SMD:R_0805_2012Metric
- SW1: value SW_SPST -> BOOT
- U3: footprint (none) -> Package_TO_SOT_SMD:SOT-223-3_TabPin2
Connections:
- net labels added: ESP_RXD0, ESP_TXD0, IO18, IO19, IO21, IO22, IO23, IO25, IO26, IO27, IO32, IO33, IO34, IO35
- net labels removed: RXD, TXD
- wire segments 25 -> 44
Other:
- moved on the sheet: J1, J2, SW1
