File: kicad_files/simpleESP32/_saved_simpleESP32.sch (KiCad schematic (older format))
At the start: 12 parts, among them J1 Conn_01x07, J2 Conn_01x07, J3 USB_B_Micro, SW1 BOOT, SW2 EN, U1 ESP32-WROOM-32D, U2 FT231XS, U3 LM1117-3.3

Commit message: finished routing
Connections:
- net +3V3: now also J1.2 (Pin_2)
- net ESP_RXD0: now also J2.4 (Pin_4)
- net ESP_TXD0: now also J2.5 (Pin_5)
- net GND: now also J1.1 (Pin_1)
- net IO18: now also J2.1 (Pin_1), U1.30 (IO18)
- net IO19: now also J2.2 (Pin_2), U1.31 (IO19)
- net IO21: now also J2.3 (Pin_3), U1.33 (IO21)
- net IO22: now also J2.6 (Pin_6), U1.36 (IO22)
- net IO23: now also J2.7 (Pin_7), U1.37 (IO23)
- net IO25: now also J1.5 (Pin_5), U1.10 (IO25)
- net IO26: now also J1.4 (Pin_4), U1.11 (IO26)
- net IO27: now also J1.3 (Pin_3), U1.12 (IO27)
- net IO32: now also J1.7 (Pin_7), U1.8 (IO32)
- net IO33: now also J1.6 (Pin_6), U1.9 (IO33)
- net at U2.13 (3V3OUT): no longer U2.3 (VCCIO)
Changed lines of the file:
@@
 Wire Wire Line
 	6000 1100 6150 1100
-Text Label 6650 4300 2    50   ~ 0
+Text Label 6650 4500 2    50   ~ 0
 ESP_TXD0
 Text Label 6650 4400 2    50   ~ 0
@@
 Wire Wire Line
 	6000 1300 6150 1300
+Text Label 6650 4700 2    50   ~ 0
+IO23
+Text Label 6650 4600 2    50   ~ 0
+IO22
+Text Label 6650 4300 2    50   ~ 0
+IO21
+Text Label 6650 4200 2    50   ~ 0
+IO19
 Text Label 6650 4100 2    50   ~ 0
-IO23
-Text Label 6650 4200 2    50   ~ 0
-IO22
-Text Label 6650 4500 2    50   ~ 0
-IO21
-Text Label 6650 4600 2    50   ~ 0
-IO19
-Text Label 6650 4700 2    50   ~ 0
 IO18
-Text Label 4500 4100 0    50   ~ 0
-IO34
-Text Label 4500 4200 0    50   ~ 0
-IO35
-Text Label 4500 4300 0    50   ~ 0
+Text Label 4500 4700 0    50   ~ 0
 IO32
-Text Label 4500 4400 0    50   ~ 0
+Text Label 4500 4600 0    50   ~ 0
 IO33
 Text Label 4500 4500 0    50   ~ 0
 IO25
-Text Label 4500 4600 0    50   ~ 0
+Text Label 4500 4400 0    50   ~ 0
 IO26
-Text Label 4500 4700 0    50   ~ 0
+Text Label 4500 4300 0    50   ~ 0
 IO27
 Text Label 3100 1500 0    50   ~ 0
@@
 Wire Wire Line
 	2850 1600 3100 1600
+$Comp
+L power:+3.3V #PWR0113
+U 1 1 5E723208
+P 4700 4200
+F 0 "#PWR0113" H 4700 4050 50  0001 C CNN
+F 1 "+3.3V" H 4715 4373 50  0000 C CNN
+F 2 "" H 4700 4200 50  0001 C CNN
+F 3 "" H 4700 4200 50  0001 C CNN
+	1    4700 4200
+	0    1    1    0
+$EndComp
+$Comp
+L power:GND #PWR0114
+U 1 1 5E7234E3
+P 4800 4000
+F 0 "#PWR0114" H 4800 3750 50  0001 C CNN
+F 1 "GND" H 4805 3827 50  0000 C CNN
+F 2 "" H 4800 4000 50  0001 C CNN
+F 3 "" H 4800 4000 50  0001 C CNN
+	1    4800 4000
+	0    -1   -1   0
+$EndComp
 Wire Wire Line
-	1450 1500 1200 1500
+	4700 4100 4700 4000
 Wire Wire Line
-	1200 1500 1200 750
+	4700 4000 4800 4000
+Text Label 6100 2600 0    50   ~ 0
+IO23
+Text Label 6100 2500 0    50   ~ 0
+IO22
+Text Label 6100 2400 0    50   ~ 0
+IO21
+Text Label 6100 2300 0    50   ~ 0
+IO19
+Text Label 6100 2200 0    50   ~ 0
+IO18
 Wire Wire Line
-	1200 750  2250 750
+	6000 2200 6100 2200
 Wire Wire Line
-	2250 750  2250 1200
+	6000 2300 6100 2300
+Wire Wire Line
+	6000 2400 6100 2400
+Wire Wire Line
+	6000 2500 6100 2500
+Wire Wire Line
+	6000 2600 6100 2600
+Text Label 6100 2700 0    50   ~ 0
+IO25
+Text Label 6100 2800 0    50   ~ 0
+IO26
+Text Label 6100 2900 0    50   ~ 0
+IO27
+Text Label 6100 3000 0    50   ~ 0
+IO32
+Wire Wire Line
+	6000 2700 6100 2700
+Wire Wire Line
+	6000 2800 6100 2800
+Wire Wire Line
+	6000 2900 6100 2900
+Wire Wire Line
+	6000 3000 6100 3000
+Text Label 6100 3100 0    50   ~ 0
+IO33
+Wire Wire Line
+	6000 3100 6100 3100
+Wire Wire Line
+	6650 4100 6750 4100
+Wire Wire Line
+	6650 4200 6750 4200
+Wire Wire Line
+	6650 4300 6750 4300
+Wire Wire Line
+	6650 4400 6750 4400
+Wire Wire Line
+	6650 4500 6750 4500
+Wire Wire Line
+	6650 4600 6750 4600
+Wire Wire Line
+	6650 4700 6750 4700
+Wire Wire Line
+	4400 4100 4700 4100
+Wire Wire Line
+	4400 4200 4700 4200
+Wire Wire Line
+	4400 4300 4500 4300
+Wire Wire Line
+	4400 4400 4500 4400
+Wire Wire Line
+	4400 4500 4500 4500
+Wire Wire Line
+	4400 4600 4500 4600
+Wire Wire Line
+	4400 4700 4500 4700
 $EndSCHEMATC
