File: kicad_files/simpleESP32/simpleESP32.kicad_pcb (KiCad board)
At the start: 2 copper layers, 23 x 46 mm, 12 parts, among them J1 Conn_01x07, J2 Conn_01x07, J3 USB_B_Micro, SW1 BOOT, SW2 EN, U1 ESP32-WROOM-32D, U2 FT231XS, U3 LM1117-3.3

Commit message: began routing
Routing:
- net +3V3: track 0.00 -> 29.5 mm
Other:
- net class Default: clearance 0.2 -> 0.1524
- rule trace_clearance: 0.2 -> 0.1524
- rule trace_min: 0.2 -> 0.153
Changed lines of the file:
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@@
     (thickness 1.6)
     (drawings 4)
-    (tracks 0)
+    (tracks 7)
     (zones 0)
     (modules 12)
@@
   )
   (setup
-    (last_trace_width 0.25)
-    (trace_clearance 0.2)
+    (last_trace_width 0.153)
+    (user_trace_width 0.153)
+    (trace_clearance 0.1524)
     (zone_clearance 0.508)
     (zone_45_only no)
-    (trace_min 0.2)
+    (trace_min 0.153)
     (segment_width 0.2)
     (edge_width 0.2)
@@
   (net 67 "Net-(U2-Pad19)")
   (net_class Default "This is the default net class."
-    (clearance 0.2)
+    (clearance 0.1524)
     (trace_width 0.25)
     (via_dia 0.8)
@@
   (gr_line (start 139 97) (end 162 97) (layer Edge.Cuts) (width 0.2))
   (gr_line (start 139 143) (end 139 97) (layer Edge.Cuts) (width 0.2))
+  (segment (start 142 99.515) (end 143.515 99.515) (width 0.153) (layer F.Cu) (net 3))
+  (segment (start 143.515 99.515) (end 143.75 99.75) (width 0.153) (layer F.Cu) (net 3))
+  (segment (start 143.75 120.6875) (end 145.5 122.4375) (width 0.153) (layer F.Cu) (net 3))
+  (segment (start 143.75 99.75) (end 143.75 120.6875) (width 0.153) (layer F.Cu) (net 3))
+  (segment (start 145.5 122.4375) (end 146.5625 122.4375) (width 0.153) (layer F.Cu) (net 3))
+  (segment (start 147.5 121.5) (end 149.35 121.5) (width 0.153) (layer F.Cu) (net 3))
+  (segment (start 146.5625 122.4375) (end 147.5 121.5) (width 0.153) (layer F.Cu) (net 3))
 )

Commit message: more routing progress
Routing:
- net /ESP_RXD0: track 0.00 -> 55.6 mm
- net /ESP_TXD0: track 0.00 -> 32.1 mm
- net Net-(SW1-Pad1): track 0.00 -> 26.0 mm
- net Net-(R1-Pad1): track 0.00 -> 24.1 mm, vias 0 -> 2
- net +3V3: track 29.5 -> 48.0 mm, vias 0 -> 2
- net +5V: track 0.00 -> 12.7 mm
- net GND: track 0.00 -> 7.10 mm
- net Net-(U2-Pad13): track 0.00 -> 6.52 mm
- net (no net): track 0.00 -> 1.33 mm
- added copper zone on B.Cu, net GND
- added copper zone on F.Cu, net GND
Changed lines of the file:
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@@
     (thickness 1.6)
     (drawings 4)
-    (tracks 7)
+    (tracks 76)
     (zones 0)
     (modules 12)
@@
   (page A4)
   (layers
-    (0 F.Cu signal)
+    (0 F.Cu signal hide)
     (31 B.Cu signal)
     (32 B.Adhes user)
@@
   (gr_line (start 139 97) (end 162 97) (layer Edge.Cuts) (width 0.2))
   (gr_line (start 139 143) (end 139 97) (layer Edge.Cuts) (width 0.2))
+  (segment (start 152.2 131.9) (end 152.2 132) (width 0.153) (layer F.Cu) (net 0))
+  (segment (start 152.2 132) (end 152.9 132.7) (width 0.153) (layer F.Cu) (net 0))
+  (segment (start 153 132.7) (end 153 132.6) (width 0.153) (layer F.Cu) (net 0))
+  (segment (start 152.9 132.7) (end 153 132.6) (width 0.153) (layer F.Cu) (net 0))
+  (segment (start 149.35 129.581914) (end 149.35 123.8) (width 0.153) (layer F.Cu) (net 1))
+  (segment (start 149.35 131.6305) (end 149.35 129.581914) (width 0.153) (layer F.Cu) (net 1))
+  (segment (start 149.857 132.1375) (end 149.35 131.6305) (width 0.153) (layer F.Cu) (net 1))
+  (segment (start 150.61 132.1375) (end 149.857 132.1375) (width 0.153) (layer F.Cu) (net 1))
+  (segment (start 151.363 132.1375) (end 153.2425 134.017) (width 0.153) (layer F.Cu) (net 1))
+  (segment (start 153.2425 134.017) (end 153.2425 134.02) (width 0.153) (layer F.Cu) (net 1))
+  (segment (start 150.61 132.1375) (end 151.363 132.1375) (width 0.153) (layer F.Cu) (net 1))
+  (segment (start 144.0625 132.1375) (end 144.1 132.1375) (width 0.153) (layer F.Cu) (net 2))
+  (segment (start 145.41 132.1375) (end 144.1 132.1375) (width 0.153) (layer F.Cu) (net 2))
+  (segment (start 151.8 131.5) (end 151.9 131.5) (width 0.153) (layer F.Cu) (net 2))
+  (segment (start 151.7975 131.5025) (end 151.8 131.5) (width 0.153) (layer F.Cu) (net 2))
+  (segment (start 150.61 131.5025) (end 151.9 131.5) (width 0.153) (layer F.Cu) (net 2))
+  (segment (start 152.3 138.5375) (end 152.3 137.7095) (width 0.153) (layer F.Cu) (net 2))
+  (segment (start 152.3 137.3) (end 152.4 137.3) (width 0.153) (layer F.Cu) (net 2))
+  (segment (start 152.3 137.7095) (end 152.4 137.3) (width 0.153) (layer F.Cu) (net 2))
+  (segment (start 144.785 116.908) (end 144.785 115.755) (width 0.153) (layer F.Cu) (net 2))
+  (segment (start 145.377 117.5) (end 144.785 116.908) (width 0.153) (layer F.Cu) (net 2))
+  (segment (start 146.4 117.5) (end 145.377 117.5) (width 0.153) (layer F.Cu) (net 2))
   (segment (start 142 99.515) (end 143.515 99.515) (width 0.153) (layer F.Cu) (net 3))
   (segment (start 143.515 99.515) (end 143.75 99.75) (width 0.153) (layer F.Cu) (net 3))
@@
   (segment (start 147.5 121.5) (end 149.35 121.5) (width 0.153) (layer F.Cu) (net 3))
   (segment (start 146.5625 122.4375) (end 147.5 121.5) (width 0.153) (layer F.Cu) (net 3))
+  (segment (start 149.35 121.5) (end 155.65 121.5) (width 0.153) (layer F.Cu) (net 3))
+  (segment (start 153.3025 128.56) (end 153.4425 128.42) (width 0.153) (layer F.Cu) (net 3))
+  (segment (start 153.3025 131.3) (end 153.3025 128.56) (width 0.153) (layer F.Cu) (net 3))
+  (via (at 156.2 126.8) (size 0.8) (drill 0.4) (layers F.Cu B.Cu) (net 3))
+  (segment (start 153.4425 128.42) (end 155.0625 126.8) (width 0.153) (layer F.Cu) (net 3))
+  (segment (start 155.0625 126.8) (end 156.2 126.8) (width 0.153) (layer F.Cu) (net 3))
+  (via (at 155.3 124.9) (size 0.8) (drill 0.4) (layers F.Cu B.Cu) (net 3))
+  (segment (start 156.2 126.8) (end 156.2 125.8) (width 0.153) (layer B.Cu) (net 3))
+  (segment (start 156.2 125.8) (end 155.3 124.9) (width 0.153) (layer B.Cu) (net 3))
+  (segment (start 155.3 121.85) (end 155.65 121.5) (width 0.153) (layer F.Cu) (net 3))
+  (segment (start 155.3 124.9) (end 155.3 121.85) (width 0.153) (layer F.Cu) (net 3))
+  (via (at 139.93 100.81) (size 0.8) (drill 0.4) (layers F.Cu B.Cu) (net 22))
+  (segment (start 142 100.785) (end 140.847 100.785) (width 0.153) (layer F.Cu) (net 22))
+  (segment (start 140.822 100.81) (end 139.93 100.81) (width 0.153) (layer F.Cu) (net 22))
+  (segment (start 140.847 100.785) (end 140.822 100.81) (width 0.153) (layer F.Cu) (net 22))
+  (via (at 145.39 118.34) (size 0.8) (drill 0.4) (layers F.Cu B.Cu) (net 22))
+  (segment (start 139.93 100.81) (end 139.93 112.88) (width 0.153) (layer B.Cu) (net 22))
+  (segment (start 139.93 112.88) (end 145.39 118.34) (width 0.153) (layer B.Cu) (net 22))
+  (segment (start 145.39 120.4525) (end 145.5 120.5625) (width 0.153) (layer F.Cu) (net 22))
+  (segment (start 145.39 118.34) (end 145.39 120.4525) (width 0.153) (layer F.Cu) (net 22))
+  (segment (start 160.2 138.497) (end 161.1 137.597) (width 0.153) (layer F.Cu) (net 23))
+  (segment (start 160.2 139.5) (end 160.2 138.497) (width 0.153) (layer F.Cu) (net 23))
+  (segment (start 161.1 117.458) (end 159 115.358) (width 0.153) (layer F.Cu) (net 23))
+  (segment (start 159 115.358) (end 159 114.755) (width 0.153) (layer F.Cu) (net 23))
+  (segment (start 161.1 137.597) (end 161.1 117.458) (width 0.153) (layer F.Cu) (net 23))
+  (segment (start 155.1 137) (end 155.1 138.9) (width 0.153) (layer F.Cu) (net 52))
+  (segment (start 147.515245 139.7) (end 146.8 138.984755) (width 0.153) (layer F.Cu) (net 52))
+  (segment (start 158.45 103.325) (end 157.478901 104.296099) (width 0.153) (layer F.Cu) (net 52))
+  (segment (start 159 103.325) (end 158.45 103.325) (width 0.153) (layer F.Cu) (net 52))
+  (segment (start 157.478901 104.296099) (end 157.478901 134.621099) (width 0.153) (layer F.Cu) (net 52))
+  (segment (start 146.8 131.5045) (end 146.163 130.8675) (width 0.153) (layer F.Cu) (net 52))
+  (segment (start 157.478901 134.621099) (end 155.1 137) (width 0.153) (layer F.Cu) (net 52))
+  (segment (start 146.163 130.8675) (end 145.41 130.8675) (width 0.153) (layer F.Cu) (net 52))
+  (segment (start 146.8 138.984755) (end 146.8 131.5045) (width 0.153) (layer F.Cu) (net 52))
+  (segment (start 154.3 139.7) (end 147.515245 139.7) (width 0.153) (layer F.Cu) (net 52))
+  (segment (start 155.1 138.9) (end 154.3 139.7) (width 0.153) (layer F.Cu) (net 52))
+  (segment (start 154.2255 126.1) (end 151.363 128.9625) (width 0.153) (layer F.Cu) (net 53))
+  (segment (start 151.363 128.9625) (end 150.61 128.9625) (width 0.153) (layer F.Cu) (net 53))
+  (segment (start 155.8 126.1) (end 154.2255 126.1) (width 0.153) (layer F.Cu) (net 53))
+  (segment (start 156.994589 124.905411) (end 155.8 126.1) (width 0.153) (layer F.Cu) (net 53))
+  (segment (start 158.45 102.055) (end 156.994589 103.510411) (width 0.153) (layer F.Cu) (net 53))
+  (segment (start 159 102.055) (end 158.45 102.055) (width 0.153) (layer F.Cu) (net 53))
+  (segment (start 156.994589 103.510411) (end 156.994589 124.905411) (width 0.153) (layer F.Cu) (net 53))
+  (segment (start 149.857 133.4075) (end 150.61 133.4075) (width 0.153) (layer F.Cu) (net 63))
+  (segment (start 145.41 130.2325) (end 146.163 130.2325) (width 0.153) (layer F.Cu) (net 63))
+  (segment (start 149.338 133.4075) (end 149.857 133.4075) (width 0.153) (layer F.Cu) (net 63))
+  (segment (start 146.163 130.2325) (end 149.338 133.4075) (width 0.153) (layer F.Cu) (net 63))
+  (zone (net 2) (net_name GND) (layer F.Cu) (hatch edge 0.508)
+    (connect_pads (clearance 0.508))
+    (min_thickness 0.254)
+    (fill yes (arc_segments 16) (thermal_gap 0.508) (thermal_bridge_width 0.508))
+    (polygon
+      (pts
+        (xy 139 97) (xy 139 143) (xy 162 143) (xy 162 97)
+      )
+    )
+  )
+  (zone (net 2) (net_name GND) (layer B.Cu) (hatch edge 0.508)
+    (connect_pads (clearance 0.508))
+    (min_thickness 0.254)
+    (fill yes (arc_segments 16) (thermal_gap 0.508) (thermal_bridge_width 0.508))
+    (polygon
+      (pts
+        (xy 139 97) (xy 139 143) (xy 162 143) (xy 162 97)
+      )
+    )
+  )
 )

Commit message: finished routing
Parts:
- renumbered SW1 to BOOT, SW2 to EN
Connections:
- J1 pad 1: Net-(J1-Pad1) -> GND
- J1 pad 2: Net-(J1-Pad2) -> +3V3
- J1 pad 3: Net-(J1-Pad3) -> /IO27
- J1 pad 4: Net-(J1-Pad4) -> /IO26
- J1 pad 5: Net-(J1-Pad5) -> /IO25
- J1 pad 6: Net-(J1-Pad6) -> /IO33
- J1 pad 7: Net-(J1-Pad7) -> /IO32
- J2 pad 1: Net-(J2-Pad1) -> /IO18
- J2 pad 2: Net-(J2-Pad2) -> /IO19
- J2 pad 3: Net-(J2-Pad3) -> /IO21
- J2 pad 4: Net-(J2-Pad4) -> /ESP_RXD0
- J2 pad 5: Net-(J2-Pad5) -> /ESP_TXD0
- J2 pad 6: Net-(J2-Pad6) -> /IO22
- J2 pad 7: Net-(J2-Pad7) -> /IO23
- U1 pad 10: Net-(U1-Pad10) -> /IO25
- U1 pad 11: Net-(U1-Pad11) -> /IO26
- U1 pad 12: Net-(U1-Pad12) -> /IO27
- U1 pad 30: Net-(U1-Pad30) -> /IO18
- U1 pad 31: Net-(U1-Pad31) -> /IO19
- U1 pad 33: Net-(U1-Pad33) -> /IO21
- U1 pad 36: Net-(U1-Pad36) -> /IO22
- U1 pad 37: Net-(U1-Pad37) -> /IO23
- U1 pad 8: Net-(U1-Pad8) -> /IO32
- U1 pad 9: Net-(U1-Pad9) -> /IO33
- U2 pad 3: Net-(U2-Pad13) -> Net-(U2-Pad3)
Routing:
- net /IO23: track 0.00 -> 39.6 mm
- net /IO22: track 0.00 -> 35.0 mm
- net /ESP_TXD0: track 32.1 -> 66.9 mm, vias 0 -> 1
- net /IO32: track 0.00 -> 31.1 mm
- net /IO33: track 0.00 -> 27.4 mm
- net /ESP_RXD0: track 55.6 -> 82.7 mm, vias 0 -> 1
- net +3V3: track 48.0 -> 70.9 mm, vias 2 -> 6
- net /IO25: track 0.00 -> 22.6 mm
- net /IO21: track 0.00 -> 22.4 mm
- net /IO26: track 0.00 -> 18.5 mm
- net /IO19: track 0.00 -> 17.1 mm
- net /IO27: track 0.00 -> 14.4 mm
- net /IO18: track 0.00 -> 13.0 mm
- net +5V: track 12.7 -> 25.0 mm
- net Net-(J3-Pad6): track 0.00 -> 6.40 mm
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Other:
- board text added: "18"
- board text added: "19"
- board text added: "21"
- board text added: "22"
- board text added: "23"
- board text added: "25"
- board text added: "26"
- board text added: "27"
- board text added: "32"
- board text added: "33"
- board text added: "GND"
- board text added: "RX0"
- board text added: "TX0"
- board text added: "VCC"

Commit message: changed silkscreen to component vals
Parts:
- renumbered C2 to 0.1uF, R1 to 10k, C1 to 10uF, C3 to 10uF
Changed lines of the file:
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@@
     (tags capacitor)
     (attr smd)
-    (fp_text reference C1 (at 0 -1.65) (layer F.SilkS)
-      (effects (font (size 1 1) (thickness 0.15)))
+    (fp_text reference 10uF (at -0.08 -1.32) (layer F.SilkS)
+      (effects (font (size 0.6 0.6) (thickness 0.15)))
     )
     (fp_text value 10uF (at 0 1.65) (layer F.Fab)
@@
     (tags capacitor)
     (attr smd)
-    (fp_text reference C2 (at 0 -1.65) (layer F.SilkS)
-      (effects (font (size 1 1) (thickness 0.15)))
+    (fp_text reference 0.1uF (at -0.14 -1.4) (layer F.SilkS)
+      (effects (font (size 0.6 0.6) (thickness 0.15)))
     )
     (fp_text value 0.1uF (at 0 1.65) (layer F.Fab)
@@
     (tags capacitor)
     (attr smd)
-    (fp_text reference C3 (at 0 -1.65) (layer F.SilkS)
-      (effects (font (size 1 1) (thickness 0.15)))
+    (fp_text reference 10uF (at 0 -1.65) (layer F.SilkS)
+      (effects (font (size 0.6 0.6) (thickness 0.15)))
     )
     (fp_text value 10uF (at 0 1.65) (layer F.Fab)
@@
     (tags resistor)
     (attr smd)
-    (fp_text reference R1 (at 0 -1.65 270) (layer F.SilkS)
-      (effects (font (size 1 1) (thickness 0.15)))
-    )
+    (fp_text reference 10k (at 0 -1.65 270) (layer F.SilkS)
+      (effects (font (size 1 1) (thickness 0.15)))
+    )
